File: ENYA-SIMR-GTWL-PCSB.kicad_sch (KiCad schematic)
At the start: 25 parts, among them J1 PICO_BLADE_1x14_MALE_RA_SMD, J2 PICO_BLADE_1x14_MALE_RA_SMD, SW1 SKSTAJE010, SW2 SKSTAJE010, SW3 SKSTAJE010, SW4 SKSTAJE010, SW5 JS5208, SW6 JS5208, SW7 SKSTAJE010, SW8 SKSTAJE010

Commit message: adding LED decoupling cap
Parts:
- added C1: 100nF_CER_0603_50V, Capacitor_SMD:C_0603_1608Metric, symbol ENYA_Cap_Smd_50V:100nF_CER_0603_50V
Connections:
- net +5V: now also C1.1
- net GND: now also C1.2
Changed lines of the file:
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@@
+    (stroke (width 0) (type default))
+  )
+  (wire (pts (xy 256.54 125.73) (xy 256.54 127))
     (stroke (width 0) (type default))
   )
@@
   )
   (bus (pts (xy 111.76 83.82) (xy 111.76 93.98))
+    (stroke (width 0) (type default))
+  )
+  (wire (pts (xy 256.54 116.84) (xy 256.54 118.11))
     (stroke (width 0) (type default))
   )
@@
     )
   )
+  (symbol (lib_id "power:GND") (at 256.54 127 0) (unit 1)
+    (in_bom yes) (on_board yes) (dnp no) (fields_autoplaced)
+    (property "Reference" "#PWR08" (at 256.54 133.35 0)
+      (effects (font (size 1.27 1.27)) hide)
+    )
+    (property "Value" "GND" (at 256.54 130.945 0)
+      (effects (font (size 1.27 1.27)))
+    )
+    (property "Footprint" "" (at 256.54 127 0)
+      (effects (font (size 1.27 1.27)) hide)
+    )
+    (property "Datasheet" "" (at 256.54 127 0)
+      (effects (font (size 1.27 1.27)) hide)
+    )
+    (pin "1")
+    (instances
+      (project "ENYA-SIMR-GTWL-PCSB"
+        (path "/6b1a3db9-0352-475b-af94-e6d69f246eea"
+          (reference "#PWR08") (unit 1)
+        )
+      )
+    )
+  )
   (symbol (lib_id "power:GND") (at 236.22 149.86 0) (unit 1)
     (in_bom yes) (on_board yes) (dnp no) (fields_autoplaced)
@@
     )
   )
+  (symbol (lib_id "ENYA_Cap_Smd_50V:100nF_CER_0603_50V") (at 256.54 121.92 0) (unit 1)
+    (in_bom yes) (on_board yes) (dnp no) (fields_autoplaced)
+    (property "Reference" "C1" (at 259.461 119.872 0)
+      (effects (font (size 1.27 1.27)) (justify left))
+    )
+    (property "Value" "100nF_CER_0603_50V" (at 257.175 124.46 0)
+      (effects (font (size 1.27 1.27)) (justify left) hide)
+    )
+    (property "Footprint" "Capacitor_SMD:C_0603_1608Metric" (at 257.5052 125.73 0)
+      (effects (font (size 1.27 1.27)) hide)
+    )
+    (property "Datasheet" "~" (at 256.54 121.92 0)
+      (effects (font (size 1.27 1.27)) hide)
+    )
+    (property "Manufacturer" "AVX Corporation" (at 256.54 121.92 0)
+      (effects (font (size 1.27 1.27)) hide)
+    )
+    (property "Manufacturer Part Number" "06033D104MAT2A" (at 256.54 121.92 0)
+      (effects (font (size 1.27 1.27)) hide)
+    )
+    (property "Digi-Key Part Number" "478-7905-1-ND" (at 256.54 121.92 0)
+      (effects (font (size 1.27 1.27)) hide)
+    )
+    (property "Capacitance" "100nF" (at 259.461 121.92 0)
+      (effects (font (size 1.27 1.27)) (justify left))
+    )
+    (property "Voltage Rating" "50V" (at 259.461 123.968 0)
+      (effects (font (size 1.27 1.27)) (justify left))
+    )
+    (pin "1")
+    (pin "2")
+    (instances
+      (project "ENYA-SIMR-GTWL-PCSB"
+        (path "/6b1a3db9-0352-475b-af94-e6d69f246eea"
+          (reference "C1") (unit 1)
+        )
+      )
+    )
+  )
   (symbol (lib_id "power:+5V") (at 236.22 96.52 0) (unit 1)
     (in_bom yes) (on_board yes) (dnp no) (fields_autoplaced)
@@
         )
       )
+    )
+  )
+  (symbol (lib_id "power:+5V") (at 256.54 116.84 0) (unit 1)
+    (in_bom yes) (on_board yes) (dnp no) (fields_autoplaced)
+    (property "Reference" "#PWR07" (at 256.54 120.65 0)
+      (effects (font (size 1.27 1.27)) hide)
+    )
+    (property "Value" "+5V" (at 256.54 112.895 0)
+      (effects (font (size 1.27 1.27)))
+    )
+    (property "Footprint" "" (at 256.54 116.84 0)
+      (effects (font (size 1.27 1.27)) hide)
+    )
+    (property "Datasheet" "" (at 256.54 116.84 0)
+      (effects (font (size 1.27 1.27)) hide)
+    )
+    (pin "1")
+    (instances
+      (project "ENYA-SIMR-GTWL-PCSB"
+        (path "/6b1a3db9-0352-475b-af94-e6d69f246eea"
+          (reference "#PWR07") (unit 1)
+        )
+      )

Commit message: correction button matrix diode polarity
Connections:
- net BTN_ROW0: now also D3.2 (A); no longer D3.1 (K)
- net BTN_ROW1: now also D4.2 (A); no longer D4.1 (K)
- net BTN_ROW2: now also D5.2 (A); no longer D5.1 (K)
- net BTN_ROW3: now also D6.2 (A); no longer D6.1 (K)
- net BTN_ROW4: now also D7.2 (A); no longer D7.1 (K)
- net BTN_ROW5: now also D8.2 (A); no longer D8.1 (K)
- net BTN_ROW6: now also D9.2 (A); no longer D9.1 (K)
- net BTN_ROW7: now also D10.2 (A); no longer D10.1 (K)
- net at SW5.2 (LEFT), SW6.2 (LEFT): now also D7.1 (K); no longer D7.2 (A)
- net at SW5.3 (PUSH), SW6.3 (PUSH): now also D5.1 (K); no longer D5.2 (A)
- net at SW5.4 (UP), SW6.4 (UP): now also D6.1 (K); no longer D6.2 (A)
- net at SW5.5 (RIGHT), SW6.5 (RIGHT): now also D9.1 (K); no longer D9.2 (A)
- net at SW5.6 (DOWN), SW6.6 (DOWN): now also D8.1 (K); no longer D8.2 (A)
- net at SW7.2, SW8.2: now also D10.1 (K); no longer D10.2 (A)
- net at SW1.2, SW2.2: now also D3.1 (K); no longer D3.2 (A)
- net at SW3.2, SW4.2: now also D4.1 (K); no longer D4.2 (A)
Other:
- moved on the sheet: D10, D3, D4, D5, D6, D7, D8, D9
Changed lines of the file:
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@@
     )
   )
-  (symbol (lib_id "ENYA_Diode_Rectifier:1N4148W-7-F_SOD-123") (at 172.72 137.16 180) (unit 1)
+  (symbol (lib_id "ENYA_Diode_Rectifier:1N4148W-7-F_SOD-123") (at 172.72 137.16 0) (unit 1)
     (in_bom yes) (on_board yes) (dnp no)
-    (property "Reference" "D9" (at 176.53 135.89 0)
-      (effects (font (size 1.27 1.27)))
-    )
-    (property "Value" "1N4148W-7-F" (at 172.72 134.3834 0)
-      (effects (font (size 1.27 1.27)) hide)
-    )
-    (property "Footprint" "Diode_SMD:D_SOD-123" (at 172.72 132.715 0)
+    (property "Reference" "D9" (at 169.545 135.89 0)
+      (effects (font (size 1.27 1.27)))
+    )
+    (property "Value" "1N4148W-7-F" (at 172.72 139.9366 0)
+      (effects (font (size 1.27 1.27)) hide)
+    )
+    (property "Footprint" "Diode_SMD:D_SOD-123" (at 172.72 141.605 0)
       (effects (font (size 1.27 1.27)) hide)
     )
@@
     )
   )
-  (symbol (lib_id "ENYA_Diode_Rectifier:1N4148W-7-F_SOD-123") (at 165.1 76.2 180) (unit 1)
+  (symbol (lib_id "ENYA_Diode_Rectifier:1N4148W-7-F_SOD-123") (at 165.1 76.2 0) (unit 1)
     (in_bom yes) (on_board yes) (dnp no) (fields_autoplaced)
     (property "Reference" "D3" (at 165.1 71.3754 0)
@@
       (effects (font (size 1.27 1.27)))
     )
-    (property "Footprint" "Diode_SMD:D_SOD-123" (at 165.1 71.755 0)
+    (property "Footprint" "Diode_SMD:D_SOD-123" (at 165.1 80.645 0)
       (effects (font (size 1.27 1.27)) hide)
     )
@@
     )
   )
-  (symbol (lib_id "ENYA_Diode_Rectifier:1N4148W-7-F_SOD-123") (at 252.73 76.2 180) (unit 1)
+  (symbol (lib_id "ENYA_Diode_Rectifier:1N4148W-7-F_SOD-123") (at 252.73 76.2 0) (unit 1)
     (in_bom yes) (on_board yes) (dnp no) (fields_autoplaced)
     (property "Reference" "D10" (at 252.73 71.3754 0)
@@
       (effects (font (size 1.27 1.27)))
     )
-    (property "Footprint" "Diode_SMD:D_SOD-123" (at 252.73 71.755 0)
+    (property "Footprint" "Diode_SMD:D_SOD-123" (at 252.73 80.645 0)
       (effects (font (size 1.27 1.27)) hide)
     )
@@
     )
   )
-  (symbol (lib_id "ENYA_Diode_Rectifier:1N4148W-7-F_SOD-123") (at 172.72 132.08 180) (unit 1)
+  (symbol (lib_id "ENYA_Diode_Rectifier:1N4148W-7-F_SOD-123") (at 172.72 132.08 0) (unit 1)
     (in_bom yes) (on_board yes) (dnp no)
-    (property "Reference" "D7" (at 176.53 130.81 0)
-      (effects (font (size 1.27 1.27)))
-    )
-    (property "Value" "1N4148W-7-F" (at 172.72 129.3034 0)
-      (effects (font (size 1.27 1.27)) hide)
-    )
-    (property "Footprint" "Diode_SMD:D_SOD-123" (at 172.72 127.635 0)
+    (property "Reference" "D7" (at 169.545 130.81 0)
+      (effects (font (size 1.27 1.27)))
+    )
+    (property "Value" "1N4148W-7-F" (at 172.72 134.8566 0)
+      (effects (font (size 1.27 1.27)) hide)
+    )
+    (property "Footprint" "Diode_SMD:D_SOD-123" (at 172.72 136.525 0)
       (effects (font (size 1.27 1.27)) hide)
     )
@@
     )
   )
-  (symbol (lib_id "ENYA_Diode_Rectifier:1N4148W-7-F_SOD-123") (at 165.1 96.52 180) (unit 1)
+  (symbol (lib_id "ENYA_Diode_Rectifier:1N4148W-7-F_SOD-123") (at 165.1 96.52 0) (unit 1)
     (in_bom yes) (on_board yes) (dnp no) (fields_autoplaced)
     (property "Reference" "D4" (at 165.1 91.6954 0)
@@
       (effects (font (size 1.27 1.27)))
     )
-    (property "Footprint" "Diode_SMD:D_SOD-123" (at 165.1 92.075 0)
+    (property "Footprint" "Diode_SMD:D_SOD-123" (at 165.1 100.965 0)
       (effects (font (size 1.27 1.27)) hide)
     )
@@
     )
   )
-  (symbol (lib_id "ENYA_Diode_Rectifier:1N4148W-7-F_SOD-123") (at 172.72 129.54 180) (unit 1)
+  (symbol (lib_id "ENYA_Diode_Rectifier:1N4148W-7-F_SOD-123") (at 172.72 129.54 0) (unit 1)
     (in_bom yes) (on_board yes) (dnp no)
-    (property "Reference" "D6" (at 176.53 128.27 0)
-      (effects (font (size 1.27 1.27)))
-    )
-    (property "Value" "1N4148W-7-F" (at 172.72 126.7634 0)
-      (effects (font (size 1.27 1.27)) hide)
-    )
-    (property "Footprint" "Diode_SMD:D_SOD-123" (at 172.72 125.095 0)
+    (property "Reference" "D6" (at 169.545 128.27 0)
+      (effects (font (size 1.27 1.27)))
+    )
+    (property "Value" "1N4148W-7-F" (at 172.72 132.3166 0)
+      (effects (font (size 1.27 1.27)) hide)
+    )
+    (property "Footprint" "Diode_SMD:D_SOD-123" (at 172.72 133.985 0)
       (effects (font (size 1.27 1.27)) hide)
     )
@@
     )
   )
-  (symbol (lib_id "ENYA_Diode_Rectifier:1N4148W-7-F_SOD-123") (at 172.72 134.62 180) (unit 1)
+  (symbol (lib_id "ENYA_Diode_Rectifier:1N4148W-7-F_SOD-123") (at 172.72 134.62 0) (unit 1)
     (in_bom yes) (on_board yes) (dnp no)
-    (property "Reference" "D8" (at 176.53 133.35 0)
-      (effects (font (size 1.27 1.27)))
-    )
-    (property "Value" "1N4148W-7-F" (at 172.72 131.8434 0)
-      (effects (font (size 1.27 1.27)) hide)
-    )
-    (property "Footprint" "Diode_SMD:D_SOD-123" (at 172.72 130.175 0)
+    (property "Reference" "D8" (at 169.545 133.35 0)
+      (effects (font (size 1.27 1.27)))
+    )
+    (property "Value" "1N4148W-7-F" (at 172.72 137.3966 0)
+      (effects (font (size 1.27 1.27)) hide)
+    )
+    (property "Footprint" "Diode_SMD:D_SOD-123" (at 172.72 139.065 0)
       (effects (font (size 1.27 1.27)) hide)
     )
@@
     )
   )
-  (symbol (lib_id "ENYA_Diode_Rectifier:1N4148W-7-F_SOD-123") (at 172.72 127 180) (unit 1)
-    (in_bom yes) (on_board yes) (dnp no) (fields_autoplaced)
-    (property "Reference" "D5" (at 172.72 122.1754 0)
-      (effects (font (size 1.27 1.27)))
-    )
-    (property "Value" "1N4148W-7-F" (at 172.72 124.2234 0)
-      (effects (font (size 1.27 1.27)))
-    )
-    (property "Footprint" "Diode_SMD:D_SOD-123" (at 172.72 122.555 0)
-      (effects (font (size 1.27 1.27)) hide)
-    )
+  (symbol (lib_id "ENYA_Diode_Rectifier:1N4148W-7-F_SOD-123") (at 172.72 127 0) (unit 1)
+    (in_bom yes) (on_board yes) (dnp no)
+    (property "Reference" "D5" (at 169.545 125.73 0)
+      (effects (font (size 1.27 1.27)))
+    )
+    (property "Value" "1N4148W-7-F" (at 172.72 123.825 0)
+      (effects (font (size 1.27 1.27)))
+    )
+    (property "Footprint" "Diode_SMD:D_SOD-123" (at 172.72 131.445 0)
+      (effects (font (size 1.27 1.27)) hide)
+    )
